Commit message: create xacro urdf file and launch file

File: ros2_study_ws/src/my_robot_description/urdf/my_robot_urdf copy.xacro (robot description, xacro)
@@ -1,4 +1,6 @@
 <?xml version="1.0"?>
-<robot name="autonomous_robot">
+<robot xmlns:xacro="http://www.ros.org/wiki/xacro" name="autonomous_robot" >
+  <xacro:property name="wheel_radius" value="0.08" />
+  <xacro:property name="wheel_length" value="0.05" />
   <!-- ================= BASE ================= -->
   <link name="base_link">
@@ -31,6 +33,7 @@
   <link name="left_wheel">
     <visual>
+      <origin xyz="0 0 -0.025" rpy="0 0 0" />
       <geometry>
-        <cylinder radius="0.08" length="0.05"/>
+        <cylinder radius="${wheel_radius}" length="${wheel_length}"/>
       </geometry>
     </visual>
@@ -45,6 +48,7 @@
   <link name="right_wheel">
     <visual>
+      <origin xyz="0 0 0.025" rpy="0 0 0" />
       <geometry>
-        <cylinder radius="0.08" length="0.05"/>
+        <cylinder radius="${wheel_radius}" length="${wheel_length}"/>
       </geometry>
     </visual>
