Commit message: Add mass and inertial into urdf

File: ros2_study_ws/src/my_robot_description/urdf/my_robot_urdf.xacro (robot description, xacro)
@@ -1,68 +1,5 @@
 <?xml version="1.0"?>
 <robot xmlns:xacro="http://www.ros.org/wiki/xacro" name="autonomous_robot" >
-  <xacro:property name="base_length" value="0.6" />
-  <xacro:property name="base_width" value="0.4" />
-  <xacro:property name="base_height" value="0.2" />
-  <xacro:property name="wheel_radius" value="0.1" />
-  <xacro:property name="wheel_length" value="0.05" />
-  <material name="grey">
-    <color rgba="0.6 0.6 0.6 1"/>
-  </material>
-  <material name="blue">
-    <color rgba="0 0 0.5 1"/>
-  </material>
-  <link name="base_footprint" />
-  <link name="base_link">
-    <visual>
-      <geometry>
-        <box size="${base_length} ${base_width} ${base_height}"/>
-      </geometry>
-      <origin xyz="0 0 ${wheel_radius}" rpy="0 0 0" />
-      <material name="blue" />
-    </visual>
-  </link>
-  <xacro:macro name="wheel_link" params="prefix">
-  <link name="${prefix}_wheel_link">
-    <visual>
-      <geometry>
-        <cylinder radius="${wheel_radius}" length="${wheel_length}"/>
-      </geometry>
-      <origin xyz="0 0 0" rpy="0 0 0" />
-      <material name="grey" />
-    </visual>
-  </link>
-  </xacro:macro>
-  <xacro:wheel_link prefix="left" />
-  <xacro:wheel_link prefix="right" />
-  <link name="caster_wheel_link">
-    <visual>
-      <geometry>
-        <sphere radius="${wheel_radius / 2.0}" />
-      </geometry>
-      <origin xyz="0 0 0" rpy="0 0 0" />
-      <material name="grey" />
-    </visual>
-  </link>
-  <joint name="base_joint" type="fixed">
-    <parent link="base_footprint"/>
-    <child link="base_link"/>
-    <origin xyz="0 0 ${wheel_radius}" rpy="0 0 0"/>
-  </joint>
-  <joint name="base_left_wheel_joint" type="continuous">
-    <parent link="base_link"/>
-    <child link="left_wheel_link"/>
-    <origin xyz="${-base_length / 4.0} ${(base_width + wheel_length) / 2.0} 0" rpy="1.5708 0 0"/>
-    <axis xyz="0 1 0"/>
-  </joint>
-  <joint name="base_right_wheel_joint" type="continuous">
-    <parent link="base_link"/>
-    <child link="right_wheel_link"/>
-    <origin xyz="${-base_length / 4.0} ${-(base_width + wheel_length) / 2.0} 0" rpy="1.5708 0 0"/>
-    <axis xyz="0 1 0"/>
-  </joint>
-  <joint name="base_caster_wheel_joint" type="fixed">
-    <parent link="base_link"/>
-    <child link="caster_wheel_link"/>
-    <origin xyz="${base_length / 3.0} 0 ${-wheel_radius / 2.0}" rpy="0 0 0"/>
-  </joint>
+  <xacro:include filename="common_properties.xacro" />
+  <xacro:include filename="mobile_base.xacro" />
 </robot>
