Commit message: Add collision and inertia properties

File: ros2_study_ws/src/my_robot_description/urdf/common_properties.xacro (robot description, xacro)
@@ -16,3 +16,21 @@
     </inertial>
   </xacro:macro>
+  <xacro:macro name="cylinder_inertia" params="m r h o_xyz o_rpy" >
+    <inertial>
+      <mass value="${m}" />
+      <origin xyz="${o_xyz}" rpy="${o_rpy}" />
+      <inertia ixx="${(m/12) * (3*r*r + h*h)}" ixy="0" ixz="0"
+               iyy="${(m/12) * (3*r*r + h*h)}" iyz="0"
+               izz="${(m/2) * (r*r)}" />
+    </inertial>
+  </xacro:macro>
+  <xacro:macro name="sphere_inertia" params="m r o_xyz o_rpy" >
+    <inertial>
+      <mass value="${m}" />
+      <origin xyz="${o_xyz}" rpy="${o_rpy}" />
+      <inertia ixx="${(2/5) * m * r * r}" ixy="0" ixz="0"
+               iyy="${(2/5) * m * r * r}" iyz="0"
+               izz="${(2/5) * m * r * r}" />
+    </inertial>
+  </xacro:macro>
 </robot>

File: ros2_study_ws/src/my_robot_description/urdf/mobile_base.xacro (robot description, xacro)
@@ -15,4 +15,10 @@
       <material name="blue" />
     </visual>
+    <collision>
+      <geometry>
+        <box size="${base_length} ${base_width} ${base_height}"/>
+      </geometry>
+      <origin xyz="0 0 ${base_height / 2.0}" rpy="0 0 0" />
+    </collision>
     <xacro:box_inertia m="5.0" x="${base_length}" y="${base_width}" z="${base_height}"
                        o_xyz="0 0 ${base_height / 2.0}" o_rpy="0 0 0" />
@@ -27,4 +33,12 @@
       <material name="grey" />
     </visual>
+    <collision>
+      <geometry>
+        <cylinder radius="${wheel_radius}" length="${wheel_length}"/>
+      </geometry>
+      <origin xyz="0 0 0" rpy="${pi / 2.0} 0 0" />
+    </collision>
+    <xacro:cylinder_inertia m="1.0" r="${wheel_radius}" h="${wheel_length}"
+                            o_xyz="0 0 0" o_rpy="${pi / 2.0} 0 0" />
   </link>
   </xacro:macro>
@@ -39,4 +53,11 @@
       <material name="grey" />
     </visual>
+    <collision>
+      <geometry>
+        <sphere radius="${wheel_radius / 2.0}" />
+      </geometry>
+      <origin xyz="0 0 0" rpy="0 0 0" />
+    </collision>
+    <xacro:sphere_inertia m="0.5" r="${wheel_radius / 2.0}" o_xyz="0 0 0" o_rpy="0 0 0" />
   </link>
   <joint name="base_joint" type="fixed">

Commit message: Add a robot arm urdf xacro

File: ros2_study_ws/src/my_robot_description/urdf/common_properties.xacro (robot description, xacro)
@@ -6,4 +6,7 @@
   <material name="blue">
     <color rgba="0 0 0.5 1"/>
+  </material>
+  <material name="orange">
+    <color rgba="1.0 0.5 0 1"/>
   </material>
   <xacro:macro name="box_inertia" params="m x y z o_xyz o_rpy" >
