Commit message: Add hand_link for arm and add collision inertia

File: ros2_study_ws/src/my_robot_description/urdf/arm.xacro (robot description, xacro)
@@ -1,23 +1,76 @@
 <?xml version="1.0"?>
 <robot xmlns:xacro="http://www.ros.org/wiki/xacro" >
-    <xacro:property name="arm_length" value="0.1" />
-    <xacro:property name="arm_width" value="0.1" />
-    <xacro:property name="arm_height" value="0.02" />
+    <xacro:property name="arm_base_length" value="0.1" />
+    <xacro:property name="arm_base_width" value="0.1" />
+    <xacro:property name="arm_base_height" value="0.02" />
+    <xacro:property name="forearm_radius" value="0.02" />
+    <xacro:property name="forearm_length" value="0.3" />
+    <xacro:property name="hand_radius" value="0.02" />
+    <xacro:property name="hand_length" value="0.3" />
     <link name="arm_base_link">
         <visual>
             <geometry>
-                <box size="${arm_length} ${arm_width} ${arm_height}"/>
+                <box size="${arm_base_length} ${arm_base_width} ${arm_base_height}"/>
             </geometry>
-            <origin xyz="0 0 0" rpy="0 0 0" />
+            <origin xyz="0 0 ${arm_base_height/2}" rpy="0 0 0" />
             <material name="orange" />
         </visual>
         <collision>
             <geometry>
-                <box size="${arm_length} ${arm_width} ${arm_height}"/>
+                <box size="${arm_base_length} ${arm_base_width} ${arm_base_height}"/>
             </geometry>
-            <origin xyz="0 0 0" rpy="0 0 0" />
+            <origin xyz="0 0 ${arm_base_height/2}" rpy="0 0 0" />
         </collision>
-        <xacro:box_inertia m="1.0" x="${arm_length}" y="${arm_width}" z="${arm_height}"
-                           o_xyz="0 0 0" o_rpy="0 0 0" />
+        <xacro:box_inertia m="1.0" x="${arm_base_length}" y="${arm_base_width}" z="${arm_base_height}"
+                           o_xyz="0 0 ${arm_base_height/2}" o_rpy="0 0 0" />
     </link>
+    <link name="forearm_link">
+        <visual>
+            <geometry>
+                <cylinder radius="${forearm_radius}" length="${forearm_length}"/>
+            </geometry>
+            <origin xyz="0 0 ${forearm_length/2}" rpy="0 0 0" />
+            <material name="yellow" />
+        </visual>
+        <collision>
+            <geometry>
+                <cylinder radius="${forearm_radius}" length="${forearm_length}"/>
+            </geometry>
+            <origin xyz="0 0 ${forearm_length/2}" rpy="0 0 0" />
+        </collision>
+        <xacro:cylinder_inertia m="1.0" r="${forearm_radius}" h="${forearm_length}"
+                                o_xyz="0 0 ${forearm_length/2}" o_rpy="0 0 0" />
+    </link>
+    <link name="hand_link">
+        <visual>
+            <geometry>
+                <cylinder radius="${hand_radius}" length="${hand_length}"/>
+            </geometry>
+            <origin xyz="0 0 ${hand_length/2}" rpy="0 0 0" />
+            <material name="orange" />
+        </visual>
+        <collision>
+            <geometry>
+                <cylinder radius="${hand_radius}" length="${hand_length}"/>
+            </geometry>
+            <origin xyz="0 0 ${hand_length/2}" rpy="0 0 0" />
+            <material name="orange" />
+        </collision>
+        <xacro:cylinder_inertia m="1.0" r="${hand_radius}" h="${hand_length}"
+                                o_xyz="0 0 ${hand_length/2}" o_rpy="0 0 0" />
+    </link>
+    <joint name="arm_base_forearm_joint" type="revolute">
+        <parent link="arm_base_link" />
+        <child link="forearm_link" />
+        <origin xyz="0 0 ${arm_base_height}" rpy="0 0 0" />
+        <axis xyz="0 1 0" />
+        <limit lower="0" upper="1.57" effort="100" velocity="100"/>
+    </joint>
+    <joint name="forearm_hand_joint" type="revolute">
+        <parent link="forearm_link" />
+        <child link="hand_link" />
+        <origin xyz="0 0 ${forearm_length}" rpy="0 0 0" />
+        <axis xyz="0 1 0" />
+        <limit lower="0" upper="1.57" effort="100" velocity="100"/>
+    </joint>
 </robot>

File: ros2_study_ws/src/my_robot_description/urdf/common_properties.xacro (robot description, xacro)
@@ -9,4 +9,7 @@
   <material name="orange">
     <color rgba="1.0 0.5 0 1"/>
+  </material>
+  <material name="yellow">
+    <color rgba="1.0 1.0 0 1"/>
   </material>
   <xacro:macro name="box_inertia" params="m x y z o_xyz o_rpy" >

File: ros2_study_ws/src/my_robot_description/urdf/standalone_arm_urdf.xacro (robot description, xacro)
@@ -1,4 +1,4 @@
 <?xml version="1.0"?>
-<robot xmlns:xacro="http://www.ros.org/wiki/xacro" name="autonomous_robot" >
+<robot xmlns:xacro="http://www.ros.org/wiki/xacro" name="robot_arm" >
     <xacro:include filename="common_properties.xacro" />
     <xacro:include filename="arm.xacro" />

Commit message: Add friction and damping for robot arm

File: ros2_study_ws/src/my_robot_description/urdf/arm.xacro (robot description, xacro)
@@ -22,5 +22,5 @@
             <origin xyz="0 0 ${arm_base_height/2}" rpy="0 0 0" />
         </collision>
-        <xacro:box_inertia m="1.0" x="${arm_base_length}" y="${arm_base_width}" z="${arm_base_height}"
+        <xacro:box_inertia m="0.3" x="${arm_base_length}" y="${arm_base_width}" z="${arm_base_height}"
                            o_xyz="0 0 ${arm_base_height/2}" o_rpy="0 0 0" />
     </link>
@@ -39,5 +39,5 @@
             <origin xyz="0 0 ${forearm_length/2}" rpy="0 0 0" />
         </collision>
-        <xacro:cylinder_inertia m="1.0" r="${forearm_radius}" h="${forearm_length}"
+        <xacro:cylinder_inertia m="0.3" r="${forearm_radius}" h="${forearm_length}"
                                 o_xyz="0 0 ${forearm_length/2}" o_rpy="0 0 0" />
     </link>
@@ -57,5 +57,5 @@
             <material name="orange" />
         </collision>
-        <xacro:cylinder_inertia m="1.0" r="${hand_radius}" h="${hand_length}"
+        <xacro:cylinder_inertia m="0.3" r="${hand_radius}" h="${hand_length}"
                                 o_xyz="0 0 ${hand_length/2}" o_rpy="0 0 0" />
     </link>
@@ -66,4 +66,5 @@
         <axis xyz="0 1 0" />
         <limit lower="0" upper="1.57" effort="100" velocity="100"/>
+        <dynamics damping="0.3" friction="0.3"/>
     </joint>
     <joint name="forearm_hand_joint" type="revolute">
@@ -73,4 +74,5 @@
         <axis xyz="0 1 0" />
         <limit lower="0" upper="1.57" effort="100" velocity="100"/>
+        <dynamics damping="0.3" friction="0.3"/>
     </joint>
 </robot>
