Commit message: Add PID parameter for robot_arm and combine the autonomous vhiche and robot arm

File: ros2_study_ws/src/my_robot_description/urdf/arm_gazebo.xacro (robot description, xacro)
@@ -5,6 +5,6 @@
                 name="gz::sim::systems::JointPositionController">
                 <joint_name>arm_base_forearm_joint</joint_name>
+                <p_gain>5.0</p_gain>
         </plugin>
-        <p_gain>5.0</p_gain>
     </gazebo>
     <gazebo>
@@ -12,6 +12,6 @@
                 name="gz::sim::systems::JointPositionController">
                 <joint_name>forearm_hand_joint</joint_name>
+                <p_gain>3.0</p_gain>
         </plugin>
-        <p_gain>3.0</p_gain>
     </gazebo>
     <gazebo>

File: ros2_study_ws/src/my_robot_description/urdf/my_robot_urdf.xacro (robot description, xacro)
@@ -4,4 +4,11 @@
   <xacro:include filename="mobile_base.xacro" />
   <xacro:include filename="mobile_base_gazebo.xacro" />
+  <xacro:include filename="arm.xacro" />
+  <xacro:include filename="arm_gazebo.xacro" />
   <xacro:include filename="camera.xacro" />
+  <joint name="mobile_base_arm_joint" type="fixed">
+    <parent link="base_link"/>
+    <child link="arm_base_link"/>
+    <origin xyz="0 0 ${base_height}" rpy="0 0 0"/>
+  </joint>
 </robot>
