Commit message: robot visual appearance_V1

File: AGV_Robot_ARM/my_robot_description/urdf/arm.xacro (robot description, xacro)
@@ -1,11 +1,11 @@
 <?xml version="1.0"?>
 <robot xmlns:xacro="http://www.ros.org/wiki/xacro" >
-    <xacro:property name="arm_base_length" value="0.1" />
-    <xacro:property name="arm_base_width" value="0.1" />
-    <xacro:property name="arm_base_height" value="0.02" />
-    <xacro:property name="forearm_radius" value="0.02" />
-    <xacro:property name="forearm_length" value="0.3" />
-    <xacro:property name="hand_radius" value="0.02" />
-    <xacro:property name="hand_length" value="0.3" />
+    <xacro:property name="arm_base_length" value="0.16" />
+    <xacro:property name="arm_base_width" value="0.16" />
+    <xacro:property name="arm_base_height" value="0.06" />
+    <xacro:property name="forearm_radius" value="0.025" />
+    <xacro:property name="forearm_length" value="0.28" />
+    <xacro:property name="hand_radius" value="0.023" />
+    <xacro:property name="hand_length" value="0.24" />
     <link name="arm_base_link">
         <visual>
@@ -14,5 +14,12 @@
             </geometry>
             <origin xyz="0 0 ${arm_base_height/2}" rpy="0 0 0" />
-            <material name="orange" />
+            <material name="dark_blue" />
+        </visual>
+        <visual>
+            <geometry>
+                <box size="${arm_base_length * 0.70} ${arm_base_width * 0.70} ${arm_base_height * 0.45}"/>
+            </geometry>
+            <origin xyz="0 0 ${arm_base_height + arm_base_height * 0.25}" rpy="0 0 0" />
+            <material name="light_grey" />
         </visual>
         <collision>
@@ -31,5 +38,12 @@
             </geometry>
             <origin xyz="0 0 ${forearm_length/2}" rpy="0 0 0" />
-            <material name="yellow" />
+            <material name="dark_grey" />
+        </visual>
+        <visual>
+            <geometry>
+                <box size="${forearm_radius * 2.2} ${forearm_radius * 2.2} ${forearm_radius * 1.2}"/>
+            </geometry>
+            <origin xyz="0 0 ${forearm_length * 0.08}" rpy="0 0 0" />
+            <material name="light_grey" />
         </visual>
         <collision>
@@ -48,4 +62,11 @@
             </geometry>
             <origin xyz="0 0 ${hand_length/2}" rpy="0 0 0" />
+            <material name="dark_grey" />
+        </visual>
+        <visual>
+            <geometry>
+                <box size="${hand_radius * 2.2} ${hand_radius * 2.2} ${hand_radius * 1.2}"/>
+            </geometry>
+            <origin xyz="0 0 ${hand_length}" rpy="0 0 0" />
             <material name="orange" />
         </visual>

File: AGV_Robot_ARM/my_robot_description/urdf/common_properties.xacro (robot description, xacro)
@@ -6,4 +6,16 @@
   <material name="blue">
     <color rgba="0 0 0.5 1"/>
+  </material>
+  <material name="dark_blue">
+    <color rgba="0.08 0.16 0.34 1"/>
+  </material>
+  <material name="dark_grey">
+    <color rgba="0.25 0.25 0.28 1"/>
+  </material>
+  <material name="light_grey">
+    <color rgba="0.85 0.85 0.87 1"/>
+  </material>
+  <material name="black">
+    <color rgba="0.08 0.08 0.08 1"/>
   </material>
   <material name="orange">

File: AGV_Robot_ARM/my_robot_description/urdf/mobile_base.xacro (robot description, xacro)
@@ -1,9 +1,9 @@
 <?xml version="1.0"?>
 <robot xmlns:xacro="http://www.ros.org/wiki/xacro" >
-  <xacro:property name="base_length" value="0.6" />
-  <xacro:property name="base_width" value="0.4" />
-  <xacro:property name="base_height" value="0.2" />
-  <xacro:property name="wheel_radius" value="0.1" />
-  <xacro:property name="wheel_length" value="0.05" />
+  <xacro:property name="base_length" value="0.7" />
+  <xacro:property name="base_width" value="0.45" />
+  <xacro:property name="base_height" value="0.18" />
+  <xacro:property name="wheel_radius" value="0.10" />
+  <xacro:property name="wheel_length" value="0.06" />
   <link name="base_footprint" />
   <link name="base_link">
@@ -13,5 +13,19 @@
       </geometry>
       <origin xyz="0 0 ${base_height / 2.0}" rpy="0 0 0" />
-      <material name="blue" />
+      <material name="dark_blue" />
+    </visual>
+    <visual>
+      <geometry>
+        <box size="${base_length * 0.82} ${base_width * 0.76} ${base_height * 0.18}"/>
+      </geometry>
+      <origin xyz="0 0 ${base_height + base_height * 0.09}" rpy="0 0 0" />
+      <material name="light_grey" />
+    </visual>
+    <visual>
+      <geometry>
+        <box size="${base_length * 0.14} ${base_width * 0.90} ${base_height * 0.22}"/>
+      </geometry>
+      <origin xyz="${base_length * 0.25} 0 ${base_height * 0.60}" rpy="0 0 0" />
+      <material name="black" />
     </visual>
     <collision>
@@ -31,5 +45,12 @@
       </geometry>
       <origin xyz="0 0 0" rpy="${pi / 2.0} 0 0" />
-      <material name="grey" />
+      <material name="dark_grey" />
+    </visual>
+    <visual>
+      <geometry>
+        <cylinder radius="${wheel_radius * 0.72}" length="${wheel_length * 0.18}"/>
+      </geometry>
+      <origin xyz="0 0 0" rpy="${pi / 2.0} 0 0" />
+      <material name="light_grey" />
     </visual>
     <collision>
@@ -51,5 +72,5 @@
       </geometry>
       <origin xyz="0 0 0" rpy="0 0 0" />
-      <material name="grey" />
+      <material name="dark_grey" />
     </visual>
     <collision>
