Commit message: Setup the initial env in gazebo

File: panda_pick_and_place/src/panda_description/urdf/arm.xacro (robot description, xacro)
@@ -7,10 +7,10 @@
     <visual>
       <geometry>
-        <mesh filename="package://panda_description/meshes/visual/link0.dae"/>
-      </geometry>
-    </visual>
-    <collision>
-      <geometry>
-        <mesh filename="package://panda_description/meshes/collision/link0.obj"/>
+        <mesh filename="$(find panda_description)/meshes/visual/link0.dae"/>
+      </geometry>
+    </visual>
+    <collision>
+      <geometry>
+        <mesh filename="$(find panda_description)/meshes/collision/link0.obj"/>
       </geometry>
     </collision>
@@ -31,10 +31,10 @@
     <visual>
       <geometry>
-        <mesh filename="package://panda_description/meshes/visual/link1.dae"/>
-      </geometry>
-    </visual>
-    <collision>
-      <geometry>
-        <mesh filename="package://panda_description/meshes/collision/link1.obj"/>
+        <mesh filename="$(find panda_description)/meshes/visual/link1.dae"/>
+      </geometry>
+    </visual>
+    <collision>
+      <geometry>
+        <mesh filename="$(find panda_description)/meshes/collision/link1.obj"/>
       </geometry>
     </collision>
@@ -58,10 +58,10 @@
     <visual>
       <geometry>
-        <mesh filename="package://panda_description/meshes/visual/link2.dae"/>
-      </geometry>
-    </visual>
-    <collision>
-      <geometry>
-        <mesh filename="package://panda_description/meshes/collision/link2.obj"/>
+        <mesh filename="$(find panda_description)/meshes/visual/link2.dae"/>
+      </geometry>
+    </visual>
+    <collision>
+      <geometry>
+        <mesh filename="$(find panda_description)/meshes/collision/link2.obj"/>
       </geometry>
     </collision>
@@ -85,10 +85,10 @@
     <visual>
       <geometry>
-        <mesh filename="package://panda_description/meshes/visual/link3.dae"/>
-      </geometry>
-    </visual>
-    <collision>
-      <geometry>
-        <mesh filename="package://panda_description/meshes/collision/link3.obj"/>
+        <mesh filename="$(find panda_description)/meshes/visual/link3.dae"/>
+      </geometry>
+    </visual>
+    <collision>
+      <geometry>
+        <mesh filename="$(find panda_description)/meshes/collision/link3.obj"/>
       </geometry>
     </collision>
@@ -112,10 +112,10 @@
     <visual>
       <geometry>
-        <mesh filename="package://panda_description/meshes/visual/link4.dae"/>
-      </geometry>
-    </visual>
-    <collision>
-      <geometry>
-        <mesh filename="package://panda_description/meshes/collision/link4.obj"/>
+        <mesh filename="$(find panda_description)/meshes/visual/link4.dae"/>
+      </geometry>
+    </visual>
+    <collision>
+      <geometry>
+        <mesh filename="$(find panda_description)/meshes/collision/link4.obj"/>
       </geometry>
     </collision>
@@ -139,10 +139,10 @@
     <visual>
       <geometry>
-        <mesh filename="package://panda_description/meshes/visual/link5.dae"/>
-      </geometry>
-    </visual>
-    <collision>
-      <geometry>
-        <mesh filename="package://panda_description/meshes/collision/link5.obj"/>
+        <mesh filename="$(find panda_description)/meshes/visual/link5.dae"/>
+      </geometry>
+    </visual>
+    <collision>
+      <geometry>
+        <mesh filename="$(find panda_description)/meshes/collision/link5.obj"/>
       </geometry>
     </collision>
@@ -166,10 +166,10 @@
     <visual>
       <geometry>
-        <mesh filename="package://panda_description/meshes/visual/link6.dae"/>
-      </geometry>
-    </visual>
-    <collision>
-      <geometry>
-        <mesh filename="package://panda_description/meshes/collision/link6.obj"/>
+        <mesh filename="$(find panda_description)/meshes/visual/link6.dae"/>
+      </geometry>
+    </visual>
+    <collision>
+      <geometry>
+        <mesh filename="$(find panda_description)/meshes/collision/link6.obj"/>
       </geometry>
     </collision>
@@ -193,10 +193,10 @@
     <visual>
       <geometry>
-        <mesh filename="package://panda_description/meshes/visual/link7.dae"/>
-      </geometry>
-    </visual>
-    <collision>
-      <geometry>
-        <mesh filename="package://panda_description/meshes/collision/link7.obj"/>
+        <mesh filename="$(find panda_description)/meshes/visual/link7.dae"/>
+      </geometry>
+    </visual>
+    <collision>
+      <geometry>
+        <mesh filename="$(find panda_description)/meshes/collision/link7.obj"/>
       </geometry>
     </collision>
@@ -220,10 +220,10 @@
     <visual>
       <geometry>
-        <mesh filename="package://panda_description/meshes/visual/hand.dae"/>
-      </geometry>
-    </visual>
-    <collision>
-      <geometry>
-        <mesh filename="package://panda_description/meshes/collision/hand.obj"/>
+        <mesh filename="$(find panda_description)/meshes/visual/hand.dae"/>
+      </geometry>
+    </visual>
+    <collision>
+      <geometry>
+        <mesh filename="$(find panda_description)/meshes/collision/hand.obj"/>
       </geometry>
     </collision>
@@ -244,10 +244,10 @@
     <visual>
       <geometry>
-        <mesh filename="package://panda_description/meshes/visual/finger.dae"/>
-      </geometry>
-    </visual>
-    <collision>
-      <geometry>
-        <mesh filename="package://panda_description/meshes/collision/finger.obj"/>
+        <mesh filename="$(find panda_description)/meshes/visual/finger.dae"/>
+      </geometry>
+    </visual>
+    <collision>
+      <geometry>
+        <mesh filename="$(find panda_description)/meshes/collision/finger.obj"/>
       </geometry>
     </collision>
@@ -263,5 +263,5 @@
       <origin rpy="0 0 3.14159265359" xyz="0 0 0"/>
       <geometry>
-        <mesh filename="package://panda_description/meshes/visual/finger.dae"/>
+        <mesh filename="$(find panda_description)/meshes/visual/finger.dae"/>
       </geometry>
     </visual>
@@ -269,5 +269,5 @@
       <origin rpy="0 0 3.14159265359" xyz="0 0 0"/>
       <geometry>
-        <mesh filename="package://panda_description/meshes/collision/finger.obj"/>
+        <mesh filename="$(find panda_description)/meshes/collision/finger.obj"/>
       </geometry>
     </collision>

File: panda_pick_and_place/src/panda_description/urdf/gazebo.xacro (robot description, xacro)
@@ -1,24 +1,91 @@
 <?xml version="1.0"?>
 <robot xmlns:xacro="http://www.ros.org/wiki/xacro" name="panda">
-  <!-- ROS 2 Control -->
-  <!-- ROS 2 Humble -->
-  <gazebo>
+  <xacro:property name="PI" value="3.14159265359" />
+  <ros2_control name="RobotSystem" type="system">
+    <!-- ros2_control Gazebo -->
+    <!-- ROS 2 Humble -->
     <xacro:if value="$(arg is_ignition)">
-      <plugin filename="ign_ros2_control-system" name="ign_ros2_control::IgnitionROS2ControlPlugin">
-        <parameters>$(find panda_controller)/config/panda_controllers.yaml</parameters>
-      </plugin>
-      <plugin filename="ignition-gazebo-sensors-system" name="ignition::gazebo::systems::Sensors">
-        <render_engine>ogre2</render_engine>
-      </plugin>
+      <hardware>
+        <plugin>ign_ros2_control/IgnitionSystem</plugin>
+      </hardware>
     </xacro:if>
     <!-- ROS 2 Iron or above -->
     <xacro:unless value="$(arg is_ignition)">
-      <plugin filename="gz_ros2_control-system" name="gz_ros2_control::GazeboSimROS2ControlPlugin">
-        <parameters>$(find panda_controller)/config/panda_controllers.yaml</parameters>
-      </plugin>
-      <plugin filename="gz-sim-sensors-system" name="gz::sim::systems::Sensors">
-        <render_engine>ogre2</render_engine>
-      </plugin>
+      <hardware>
+        <plugin>gz_ros2_control/GazeboSimSystem</plugin>
+      </hardware>
     </xacro:unless>
-  </gazebo>
+    <!-- Joint 1 -->
+    <joint name="panda_joint1">
+      <command_interface name="position">
+        <param name="min">-2.9671</param>
+        <param name="max">2.9671</param>
+      </command_interface>
+      <state_interface name="position"/>
+    </joint>
+    <!-- Joint 2 -->
+    <joint name="panda_joint2">
+      <command_interface name="position">
+        <param name="min">-1.8326</param>
+        <param name="max">1.8326</param>
+      </command_interface>
+      <state_interface name="position"/>
+    </joint>
+    <!-- Joint 3 -->
+    <joint name="panda_joint3">
+      <command_interface name="position">
+        <param name="min">-2.9671</param>
+        <param name="max">2.9671</param>
+      </command_interface>
+      <state_interface name="position"/>
+    </joint>
+    <!-- Joint 4 -->
+    <joint name="panda_joint4">
+      <command_interface name="position">
+        <param name="min">-3.1416</param>
+        <param name="max">0.0</param>
+      </command_interface>
+      <state_interface name="position"/>
+    </joint>
+    <!-- Joint 5 -->
+    <joint name="panda_joint5">
+      <command_interface name="position">
+        <param name="min">-2.9671</param>
+        <param name="max">2.9671</param>
+      </command_interface>
+      <state_interface name="position"/>
+    </joint>
+    <!-- Joint 6 -->
+    <joint name="panda_joint6">
+      <command_interface name="position">
+        <param name="min">-0.0873</param>
+        <param name="max">3.8223</param>
+      </command_interface>
+      <state_interface name="position"/>
+    </joint>
+    <!-- Joint 7 -->
+    <joint name="panda_joint7">
+      <command_interface name="position">
+        <param name="min">-2.9671</param>
+        <param name="max">2.9671</param>
+      </command_interface>
+      <state_interface name="position"/>
+    </joint>
+    <!-- Gripper Finger Joint 1 -->
+    <joint name="panda_finger_joint1">
+      <command_interface name="position">
+        <param name="min">0.0</param>
+        <param name="max">0.04</param>
+      </command_interface>
+      <state_interface name="position"/>
+    </joint>
+    <!-- Gripper Finger Joint 2 (Mimics Joint 1) -->
+    <joint name="panda_finger_joint2">
+      <command_interface name="position">
+        <param name="min">0.0</param>
+        <param name="max">0.04</param>
+      </command_interface>
+      <state_interface name="position"/>
+    </joint>
+  </ros2_control>
 </robot>

File: panda_pick_and_place/src/panda_description/urdf/panda_urdf.xacro (robot description, xacro)
@@ -1,8 +1,9 @@
 <?xml version="1.0"?>
 <robot name="panda" xmlns:xacro="http://www.ros.org/wiki/xacro">
+  <xacro:arg name="is_ignition" default="false"/>
   <!-- <xacro:include filename="$(find panda_description)/urdf/materials.xacro" /> -->
   <xacro:include filename="$(find panda_description)/urdf/arm.xacro" />
   <!-- <xacro:include filename="$(find panda_description)/urdf/sensors.xacro" /> -->
   <xacro:include filename="$(find panda_description)/urdf/gazebo.xacro" />
-  <xacro:include filename="$(find panda_description)/urdf/ros2control.xacro" />
+  <!-- <xacro:include filename="$(find panda_description)/urdf/ros2_control.xacro" /> -->
 </robot>

File: panda_pick_and_place/src/panda_description/urdf/ros2_control.xacro (robot description, xacro)
@@ -1,91 +1,24 @@
 <?xml version="1.0"?>
 <robot xmlns:xacro="http://www.ros.org/wiki/xacro" name="panda">
-  <xacro:property name="PI" value="3.14159265359" />
-  <ros2_control name="RobotSystem" type="system">
-    <!-- ros2_control Gazebo -->
-    <!-- ROS 2 Humble -->
+  <!-- ROS 2 Control -->
+  <!-- ROS 2 Humble -->
+  <gazebo>
     <xacro:if value="$(arg is_ignition)">
-      <hardware>
-        <plugin>ign_ros2_control/IgnitionSystem</plugin>
-      </hardware>
+      <plugin filename="ign_ros2_control-system" name="ign_ros2_control::IgnitionROS2ControlPlugin">
+        <parameters>$(find panda_controller)/config/panda_controllers.yaml</parameters>
+      </plugin>
+      <plugin filename="ignition-gazebo-sensors-system" name="ignition::gazebo::systems::Sensors">
+        <render_engine>ogre2</render_engine>
+      </plugin>
     </xacro:if>
     <!-- ROS 2 Iron or above -->
     <xacro:unless value="$(arg is_ignition)">
-      <hardware>
-        <plugin>gz_ros2_control/GazeboSimSystem</plugin>
-      </hardware>
+      <plugin filename="gz_ros2_control-system" name="gz_ros2_control::GazeboSimROS2ControlPlugin">
+        <parameters>$(find panda_controller)/config/panda_controllers.yaml</parameters>
+      </plugin>
+      <plugin filename="gz-sim-sensors-system" name="gz::sim::systems::Sensors">
+        <render_engine>ogre2</render_engine>
+      </plugin>
     </xacro:unless>
-    <!-- Joint 1 -->
-    <joint name="panda_joint1">
-      <command_interface name="position">
-        <param name="min">-2.9671</param>
-        <param name="max">2.9671</param>
-      </command_interface>
-      <state_interface name="position"/>
-    </joint>
-    <!-- Joint 2 -->
-    <joint name="panda_joint2">
-      <command_interface name="position">
-        <param name="min">-1.8326</param>
-        <param name="max">1.8326</param>
-      </command_interface>
-      <state_interface name="position"/>
-    </joint>
-    <!-- Joint 3 -->
-    <joint name="panda_joint3">
-      <command_interface name="position">
-        <param name="min">-2.9671</param>
-        <param name="max">2.9671</param>
-      </command_interface>
-      <state_interface name="position"/>
-    </joint>
-    <!-- Joint 4 -->
-    <joint name="panda_joint4">
-      <command_interface name="position">
-        <param name="min">-3.1416</param>
-        <param name="max">0.0</param>
-      </command_interface>
-      <state_interface name="position"/>
-    </joint>
-    <!-- Joint 5 -->
-    <joint name="panda_joint5">
-      <command_interface name="position">
-        <param name="min">-2.9671</param>
-        <param name="max">2.9671</param>
-      </command_interface>
-      <state_interface name="position"/>
-    </joint>
-    <!-- Joint 6 -->
-    <joint name="panda_joint6">
-      <command_interface name="position">
-        <param name="min">-0.0873</param>
-        <param name="max">3.8223</param>
-      </command_interface>
-      <state_interface name="position"/>
-    </joint>
-    <!-- Joint 7 -->
-    <joint name="panda_joint7">
-      <command_interface name="position">
-        <param name="min">-2.9671</param>
-        <param name="max">2.9671</param>
-      </command_interface>
-      <state_interface name="position"/>
-    </joint>
-    <!-- Gripper Finger Joint 1 -->
-    <joint name="panda_finger_joint1">
-      <command_interface name="position">
-        <param name="min">0.0</param>
-        <param name="max">0.04</param>
-      </command_interface>
-      <state_interface name="position"/>
-    </joint>
-    <!-- Gripper Finger Joint 2 (Mimics Joint 1) -->
-    <joint name="panda_finger_joint2">
-      <command_interface name="position">
-        <param name="min">0.0</param>
-        <param name="max">0.04</param>
-      </command_interface>
-      <state_interface name="position"/>
-    </joint>
-  </ros2_control>
+  </gazebo>
 </robot>

Commit message: Fixed the bug that mesh URI not work for both MoveIt_setup_assistant and Gazebo

File: panda_pick_and_place/src/panda_description/urdf/arm.xacro (robot description, xacro)
@@ -1,4 +1,5 @@
 <?xml version="1.0" ?>
 <robot name="panda" xmlns:xacro="http://www.ros.org/wiki/xacro">
+  <xacro:arg name="mesh_prefix" default="package://panda_description/meshes"/>
   <!-- World Frame -->
   <link name="world"/>
@@ -7,10 +8,10 @@
     <visual>
       <geometry>
-        <mesh filename="$(find panda_description)/meshes/visual/link0.dae"/>
-      </geometry>
-    </visual>
-    <collision>
-      <geometry>
-        <mesh filename="$(find panda_description)/meshes/collision/link0.obj"/>
+        <mesh filename="$(arg mesh_prefix)/visual/link0.dae"/>
+      </geometry>
+    </visual>
+    <collision>
+      <geometry>
+        <mesh filename="$(arg mesh_prefix)/collision/link0.obj"/>
       </geometry>
     </collision>
@@ -31,10 +32,10 @@
     <visual>
       <geometry>
-        <mesh filename="$(find panda_description)/meshes/visual/link1.dae"/>
-      </geometry>
-    </visual>
-    <collision>
-      <geometry>
-        <mesh filename="$(find panda_description)/meshes/collision/link1.obj"/>
+        <mesh filename="$(arg mesh_prefix)/visual/link1.dae"/>
+      </geometry>
+    </visual>
+    <collision>
+      <geometry>
+        <mesh filename="$(arg mesh_prefix)/collision/link1.obj"/>
       </geometry>
     </collision>
@@ -58,10 +59,10 @@
     <visual>
       <geometry>
-        <mesh filename="$(find panda_description)/meshes/visual/link2.dae"/>
-      </geometry>
-    </visual>
-    <collision>
-      <geometry>
-        <mesh filename="$(find panda_description)/meshes/collision/link2.obj"/>
+        <mesh filename="$(arg mesh_prefix)/visual/link2.dae"/>
+      </geometry>
+    </visual>
+    <collision>
+      <geometry>
+        <mesh filename="$(arg mesh_prefix)/collision/link2.obj"/>
       </geometry>
     </collision>
@@ -85,10 +86,10 @@
     <visual>
       <geometry>
-        <mesh filename="$(find panda_description)/meshes/visual/link3.dae"/>
-      </geometry>
-    </visual>
-    <collision>
-      <geometry>
-        <mesh filename="$(find panda_description)/meshes/collision/link3.obj"/>
+        <mesh filename="$(arg mesh_prefix)/visual/link3.dae"/>
+      </geometry>
+    </visual>
+    <collision>
+      <geometry>
+        <mesh filename="$(arg mesh_prefix)/collision/link3.obj"/>
       </geometry>
     </collision>
@@ -112,10 +113,10 @@
     <visual>
       <geometry>
-        <mesh filename="$(find panda_description)/meshes/visual/link4.dae"/>
-      </geometry>
-    </visual>
-    <collision>
-      <geometry>
-        <mesh filename="$(find panda_description)/meshes/collision/link4.obj"/>
+        <mesh filename="$(arg mesh_prefix)/visual/link4.dae"/>
+      </geometry>
+    </visual>
+    <collision>
+      <geometry>
+        <mesh filename="$(arg mesh_prefix)/collision/link4.obj"/>
       </geometry>
     </collision>
@@ -139,10 +140,10 @@
     <visual>
       <geometry>
-        <mesh filename="$(find panda_description)/meshes/visual/link5.dae"/>
-      </geometry>
-    </visual>
-    <collision>
-      <geometry>
-        <mesh filename="$(find panda_description)/meshes/collision/link5.obj"/>
+        <mesh filename="$(arg mesh_prefix)/visual/link5.dae"/>
+      </geometry>
+    </visual>
+    <collision>
+      <geometry>
+        <mesh filename="$(arg mesh_prefix)/collision/link5.obj"/>
       </geometry>
     </collision>
@@ -166,10 +167,10 @@
     <visual>
       <geometry>
-        <mesh filename="$(find panda_description)/meshes/visual/link6.dae"/>
-      </geometry>
-    </visual>
-    <collision>
-      <geometry>
-        <mesh filename="$(find panda_description)/meshes/collision/link6.obj"/>
+        <mesh filename="$(arg mesh_prefix)/visual/link6.dae"/>
+      </geometry>
+    </visual>
+    <collision>
+      <geometry>
+        <mesh filename="$(arg mesh_prefix)/collision/link6.obj"/>
       </geometry>
     </collision>
@@ -193,10 +194,10 @@
     <visual>
       <geometry>
-        <mesh filename="$(find panda_description)/meshes/visual/link7.dae"/>
-      </geometry>
-    </visual>
-    <collision>
-      <geometry>
-        <mesh filename="$(find panda_description)/meshes/collision/link7.obj"/>
+        <mesh filename="$(arg mesh_prefix)/visual/link7.dae"/>
+      </geometry>
+    </visual>
+    <collision>
+      <geometry>
+        <mesh filename="$(arg mesh_prefix)/collision/link7.obj"/>
       </geometry>
     </collision>
@@ -220,10 +221,10 @@
     <visual>
       <geometry>
-        <mesh filename="$(find panda_description)/meshes/visual/hand.dae"/>
-      </geometry>
-    </visual>
-    <collision>
-      <geometry>
-        <mesh filename="$(find panda_description)/meshes/collision/hand.obj"/>
+        <mesh filename="$(arg mesh_prefix)/visual/hand.dae"/>
+      </geometry>
+    </visual>
+    <collision>
+      <geometry>
+        <mesh filename="$(arg mesh_prefix)/collision/hand.obj"/>
       </geometry>
     </collision>
@@ -244,10 +245,10 @@
     <visual>
       <geometry>
-        <mesh filename="$(find panda_description)/meshes/visual/finger.dae"/>
-      </geometry>
-    </visual>
-    <collision>
-      <geometry>
-        <mesh filename="$(find panda_description)/meshes/collision/finger.obj"/>
+        <mesh filename="$(arg mesh_prefix)/visual/finger.dae"/>
+      </geometry>
+    </visual>
+    <collision>
+      <geometry>
+        <mesh filename="$(arg mesh_prefix)/collision/finger.obj"/>
       </geometry>
     </collision>
@@ -263,5 +264,5 @@
       <origin rpy="0 0 3.14159265359" xyz="0 0 0"/>
       <geometry>
-        <mesh filename="$(find panda_description)/meshes/visual/finger.dae"/>
+        <mesh filename="$(arg mesh_prefix)/visual/finger.dae"/>
       </geometry>
     </visual>
@@ -269,5 +270,5 @@
       <origin rpy="0 0 3.14159265359" xyz="0 0 0"/>
       <geometry>
-        <mesh filename="$(find panda_description)/meshes/collision/finger.obj"/>
+        <mesh filename="$(arg mesh_prefix)/collision/finger.obj"/>
       </geometry>
     </collision>

File: panda_pick_and_place/src/panda_description/urdf/panda_urdf.xacro (robot description, xacro)
@@ -1,4 +1,5 @@
 <?xml version="1.0"?>
 <robot name="panda" xmlns:xacro="http://www.ros.org/wiki/xacro">
+  <xacro:arg name="mesh_prefix" default="package://panda_description/meshes"/>
   <xacro:arg name="is_ignition" default="false"/>
   <!-- <xacro:include filename="$(find panda_description)/urdf/materials.xacro" /> -->
