Commit message: Improve Panda Gazebo workcell environment

File: panda_pick_and_place/src/panda_description/urdf/sensors.xacro (robot description, xacro)
@@ -12,5 +12,7 @@
                 <box size="0.1 0.1 0.05"/>
             </geometry>
-            <material name="red"/>
+            <material name="red">
+                <color rgba="1 0 0 1"/>
+            </material>
         </visual>
         <collision>
@@ -19,5 +21,4 @@
                 <box size="0.1 0.1 0.05"/>
             </geometry>
-            <material name="red"/>
         </collision>
     </link>
